Commit message: added left and right tank

File: urdf/all.urdf (robot description, URDF)
Before this commit: robot custom_env, 15 links, 14 joints
Joints:
- removed joint gripper_joint
- added joint enclosure_joint: type fixed, parent tool0, child enclosure, origin xyz=0 0 0 rpy=0 0 0

File: urdf/all.xacro (robot description, xacro)
@@ -2,14 +2,10 @@
 <robot xmlns:xacro="http://www.ros.org/wiki/xacro" name="custom_env">
   <xacro:include filename="$(find ur_description)/urdf/ur10.xacro"/>
-  <xacro:include filename="$(find cgras_scene)/urdf/gripper.xacro"/>
+  <xacro:include filename="$(find cgras_scene)/urdf/enclosure.xacro"/>
   <xacro:include filename="$(find cgras_scene)/urdf/trolley.xacro"/>
   <xacro:include filename="$(find cgras_scene)/urdf/tank.xacro"/>
-  <!--
-  <xacro:include filename="$(find armer_descriptions)/data/custom/cgras_descriptions/robots/tank_right.xacro"/>
-  <xacro:include filename="$(find armer_descriptions)/data/custom/cgras_descriptions/robots/tank_left.xacro"/>
-  -->
-  <xacro:gripper xyz="0 0 0" rpy="0 0 0" connected_to="tool0" />
-  <!-- <xacro:xarm_device dof="6" /> -->
-  <!-- <xacro:gripper xyz="0 0 0" rpy="0 0 ${pi/2}" connected_to="link_eef" /> -->
+  <xacro:include filename="$(find cgras_scene)/urdf/tank_left.xacro"/>
+  <xacro:include filename="$(find cgras_scene)/urdf/tank_right.xacro"/>
+  <xacro:enclosure xyz="0 0 0" rpy="0 0 0" connected_to="tool0" />
   <xacro:trolley rpy="0 0 ${pi/2}" connected_to="base_link" />
   <!-- <xacro:tank xyz="0 0 0" rpy="0 0 ${pi/2}" connected_to="base_link" /> -->

File: urdf/enclosure.xacro (robot description, xacro)
@@ -1,7 +1,7 @@
 <?xml version="1.0" encoding="utf-8"?>
-<robot xmlns:xacro="http://www.ros.org/wiki/xacro" name="gripper">
-  <xacro:macro name="gripper" params="connected_to:='' rpy:='0 0 0' xyz:='0 0 0'">
+<robot xmlns:xacro="http://www.ros.org/wiki/xacro" name="enclosure">
+  <xacro:macro name="enclosure" params="connected_to:='' rpy:='0 0 0' xyz:='0 0 0'">
     <xacro:unless value="${connected_to == ''}">
-      <joint name="gripper_joint" type="fixed">
+      <joint name="enclosure_joint" type="fixed">
         <parent link="${connected_to}"/>
         <child link="enclosure"/>
@@ -44,7 +44,7 @@
       </collision>
     </link> -->
-    <!-- Gripper Joint Definitions (Includes Framos Model Individually)-->
+    <!-- enclosure Joint Definitions (Includes Framos Model Individually)-->
     <!-- <joint name="framos_joint" type="fixed">
-      <parent link="gripper_link"/>
+      <parent link="enclosure"/>
       <child link="framos_link"/>
       <origin xyz="0 -0.02657 0.096" rpy="0 0 0"/>

File: urdf/tank.xacro (robot description, xacro)
@@ -27,5 +27,5 @@
         <origin xyz="0 0 0" rpy="0 0 0"/>
         <geometry>
-          <mesh filename="package://cgras_scene/meshes/visual/Settlement_Centred.stl" scale="0.001 0.001 0.001"/>
+          <mesh filename="package://cgras_scene/meshes/visual/SettlementSystem.stl" scale="0.001 0.001 0.001"/>
         </geometry>
       </visual>
@@ -33,5 +33,5 @@
         <origin xyz="0 0 0" rpy="0 0 0"/>
         <geometry>
-          <mesh filename="package://cgras_scene/meshes/collision/Settlement_Centred.stl" scale="0.001 0.001 0.001"/>
+          <mesh filename="package://cgras_scene/meshes/collision/SettlementSystem.stl" scale="0.001 0.001 0.001"/>
         </geometry>
       </collision>

Commit message: test add mesh

File: urdf/all.urdf (robot description, URDF)
Before this commit: robot custom_env, 15 links, 14 joints
Joints:
- joint robot_base_to_robot_joint: origin xyz=0 0 0 rpy=0 0 1.5707963267948966 -> xyz=0 0 0 rpy=0 0 0

File: urdf/all.xacro (robot description, xacro)
@@ -8,11 +8,9 @@
   <xacro:include filename="$(find cgras_scene)/urdf/tank_right.xacro"/>
   <xacro:enclosure xyz="0 0 0" rpy="0 0 0" connected_to="tool0" />
-  <xacro:trolley rpy="0 0 ${pi/2}" connected_to="base_link" />
-  <!-- <xacro:tank xyz="0 0 0" rpy="0 0 ${pi/2}" connected_to="base_link" /> -->
+  <xacro:trolley rpy="0 0 0" connected_to="base_link" />
 <!--
-  <xacro:tank_right xyz="0 0 0" rpy="0 0 0" connected_to="base_link" />
+  <xacro:tank_right xyz="0 -0.45 1.1" rpy="0 0 -${pi/2}" connected_to="trolley" />
   <xacro:tank_left xyz="0 0 0" rpy="0 0 0" connected_to="base_link" />
-  -->
-  <!-- <xacro:tank xyz="-0.5 0.75 0" rpy="${-pi/2} 0 ${pi/2}" connected_to="base_link" /> -->
+  <xacro:tank xyz="-0.5 0.75 0" rpy="${-pi/2} 0 ${pi/2}" connected_to="base_link" /> -->
 <!--
   <link name="world" />

File: urdf/tank_right.xacro (robot description, xacro)
@@ -42,5 +42,5 @@
       <parent link="tank_right_tag"/>
       <child link="tank_right_tag_mount"/>
-      <origin xyz="0.014 0 -0.082" rpy="0 ${pi/2} 0"/>
+      <origin xyz="0.014 0 -0.082" rpy="0 0 0"/>
     </joint>
     <!-- Where the tag is on the tank -->
@@ -48,5 +48,5 @@
       <parent link="tank_right_tag_mount"/>
       <child link="tank_right"/>
-      <origin xyz="0.415 -0.0685 -1.075" rpy="0 0 0"/>
+      <origin xyz="0.41 0.06 -1.080" rpy="0 0 0"/>
     </joint>
   </xacro:macro>
